Commit message: Auto-update: 2026-04-12 23:00

File: src/ammr_bringup/urdf/ammr_base.urdf.xacro (robot description, xacro)
@@ -142,4 +142,45 @@
     </inertial>
   </link>
+  <!-- ===== LiDAR link ===== -->
+  <joint name="lidar_joint" type="fixed">
+    <parent link="base_link"/>
+    <child  link="lidar_link"/>
+    <origin xyz="0 0 ${base_height/2 + 0.05}" rpy="0 0 0"/>
+  </joint>
+  <link name="lidar_link">
+    <visual>
+      <geometry><cylinder radius="0.05" length="0.04"/></geometry>
+      <material name="black2"><color rgba="0.1 0.1 0.1 1.0"/></material>
+    </visual>
+    <inertial>
+      <mass value="0.1"/>
+      <inertia ixx="0.0001" ixy="0" ixz="0" iyy="0.0001" iyz="0" izz="0.0001"/>
+    </inertial>
+  </link>
+  <!-- Gazebo LiDAR sensor -->
+  <gazebo reference="lidar_link">
+    <sensor name="lidar" type="gpu_lidar">
+      <pose>0 0 0 0 0 0</pose>
+      <topic>/scan</topic>
+      <update_rate>10</update_rate>
+      <ray>
+        <scan>
+          <horizontal>
+            <samples>360</samples>
+            <resolution>1</resolution>
+            <min_angle>-3.14159</min_angle>
+            <max_angle>3.14159</max_angle>
+          </horizontal>
+        </scan>
+        <range>
+          <min>0.12</min>
+          <max>10.0</max>
+          <resolution>0.01</resolution>
+        </range>
+      </ray>
+      <always_on>true</always_on>
+      <visualize>true</visualize>
+    </sensor>
+  </gazebo>
   <!-- ===== Gazebo diff-drive plugin ===== -->
   <gazebo>

Commit message: Auto-update: 2026-04-15 17:02

File: src/ammr_bringup/urdf/ammr_base.urdf.xacro (robot description, xacro)
@@ -1,10 +1,11 @@
 <?xml version="1.0"?>
 <robot name="ammr_base" xmlns:xacro="http://www.ros.org/wiki/xacro">
-  <!-- Properties -->
-  <xacro:property name="base_size"    value="0.4"/>
+  <!-- Properties：60cm 直徑圓形底盤 + 4 差速輪 -->
+  <xacro:property name="base_radius"  value="0.30"/>   <!-- 60cm 直徑 -->
   <xacro:property name="base_height"  value="0.12"/>
   <xacro:property name="wheel_radius" value="0.08"/>
-  <xacro:property name="wheel_width"  value="0.04"/>
-  <xacro:property name="wheel_offset" value="0.22"/>  <!-- distance from center to wheel -->
+  <xacro:property name="wheel_width"  value="0.05"/>
+  <xacro:property name="wheel_x"      value="0.13"/>   <!-- 前後輪距中心距離 -->
+  <xacro:property name="wheel_y"      value="0.24"/>   <!-- 左右輪距中心距離 -->
   <!-- base_footprint -->
   <link name="base_footprint"/>
@@ -14,9 +15,9 @@
     <origin xyz="0 0 ${wheel_radius}" rpy="0 0 0"/>
   </joint>
-  <!-- Body -->
+  <!-- 圓形底盤本體 -->
   <link name="base_link">
     <visual>
       <geometry>
-        <box size="${base_size} ${base_size} ${base_height}"/>
+        <cylinder radius="${base_radius}" length="${base_height}"/>
       </geometry>
       <material name="blue">
@@ -26,120 +27,50 @@
     <collision>
       <geometry>
-        <box size="${base_size} ${base_size} ${base_height}"/>
+        <cylinder radius="${base_radius}" length="${base_height}"/>
       </geometry>
     </collision>
     <inertial>
-      <mass value="8.0"/>
-      <inertia ixx="0.13" ixy="0.0" ixz="0.0"
-                           iyy="0.13" iyz="0.0"
-                                      izz="0.22"/>
+      <mass value="15.0"/>
+      <!-- 實心圓柱慣性矩 -->
+      <inertia ixx="0.356" ixy="0.0" ixz="0.0"
+                           iyy="0.356" iyz="0.0"
+                                       izz="0.675"/>
     </inertial>
   </link>
-  <!-- ===== LEFT wheel (active, diff-drive) ===== -->
-  <joint name="left_wheel_joint" type="continuous">
-    <parent link="base_link"/>
-    <child  link="left_wheel"/>
-    <origin xyz="0 ${wheel_offset} ${-base_height/2}" rpy="${-pi/2} 0 0"/>
-    <axis xyz="0 0 1"/>
-  </joint>
-  <link name="left_wheel">
-    <visual>
-      <geometry>
-        <cylinder radius="${wheel_radius}" length="${wheel_width}"/>
-      </geometry>
-      <material name="dark">
-        <color rgba="0.1 0.1 0.1 1.0"/>
-      </material>
-    </visual>
-    <collision>
-      <geometry>
-        <cylinder radius="${wheel_radius}" length="${wheel_width}"/>
-      </geometry>
-    </collision>
-    <inertial>
-      <mass value="0.5"/>
-      <inertia ixx="0.001" ixy="0.0" ixz="0.0"
-                           iyy="0.001" iyz="0.0"
-                                       izz="0.002"/>
-    </inertial>
-  </link>
-  <!-- ===== RIGHT wheel (active, diff-drive) ===== -->
-  <joint name="right_wheel_joint" type="continuous">
-    <parent link="base_link"/>
-    <child  link="right_wheel"/>
-    <origin xyz="0 ${-wheel_offset} ${-base_height/2}" rpy="${-pi/2} 0 0"/>
-    <axis xyz="0 0 1"/>
-  </joint>
-  <link name="right_wheel">
-    <visual>
-      <geometry>
-        <cylinder radius="${wheel_radius}" length="${wheel_width}"/>
-      </geometry>
-      <material name="dark"/>
-    </visual>
-    <collision>
-      <geometry>
-        <cylinder radius="${wheel_radius}" length="${wheel_width}"/>
-      </geometry>
-    </collision>
-    <inertial>
-      <mass value="0.5"/>
-      <inertia ixx="0.001" ixy="0.0" ixz="0.0"
-                           iyy="0.001" iyz="0.0"
-                                       izz="0.002"/>
-    </inertial>
-  </link>
-  <!-- ===== FRONT caster (passive) ===== -->
-  <joint name="front_caster_joint" type="fixed">
-    <parent link="base_link"/>
-    <child  link="front_caster"/>
-    <origin xyz="${wheel_offset} 0 ${-base_height/2 - wheel_radius/2}" rpy="0 0 0"/>
-  </joint>
-  <link name="front_caster">
-    <visual>
-      <geometry>
-        <sphere radius="${wheel_radius/2}"/>
-      </geometry>
-      <material name="grey">
-        <color rgba="0.5 0.5 0.5 1.0"/>
-      </material>
-    </visual>
-    <collision>
-      <geometry>
-        <sphere radius="${wheel_radius/2}"/>
-      </geometry>
-    </collision>
-    <inertial>
-      <mass value="0.1"/>
-      <inertia ixx="0.0001" ixy="0.0" ixz="0.0"
-                            iyy="0.0001" iyz="0.0"
-                                         izz="0.0001"/>
-    </inertial>
-  </link>
-  <!-- ===== BACK caster (passive) ===== -->
-  <joint name="back_caster_joint" type="fixed">
-    <parent link="base_link"/>
-    <child  link="back_caster"/>
-    <origin xyz="${-wheel_offset} 0 ${-base_height/2 - wheel_radius/2}" rpy="0 0 0"/>
-  </joint>
-  <link name="back_caster">
-    <visual>
-      <geometry>
-        <sphere radius="${wheel_radius/2}"/>
-      </geometry>
-      <material name="grey"/>
-    </visual>
-    <collision>
-      <geometry>
-        <sphere radius="${wheel_radius/2}"/>
-      </geometry>
-    </collision>
-    <inertial>
-      <mass value="0.1"/>
-      <inertia ixx="0.0001" ixy="0.0" ixz="0.0"
-                            iyy="0.0001" iyz="0.0"
-                                         izz="0.0001"/>
-    </inertial>
-  </link>
+  <!-- ===== 輪子 xacro macro ===== -->
+  <xacro:macro name="wheel" params="name x y">
+    <joint name="${name}_joint" type="continuous">
+      <parent link="base_link"/>
+      <child  link="${name}"/>
+      <origin xyz="${x} ${y} ${-base_height/2}" rpy="${-pi/2} 0 0"/>
+      <axis xyz="0 0 1"/>
+    </joint>
+    <link name="${name}">
+      <visual>
+        <geometry>
+          <cylinder radius="${wheel_radius}" length="${wheel_width}"/>
+        </geometry>
+        <material name="dark">
+          <color rgba="0.1 0.1 0.1 1.0"/>
+        </material>
+      </visual>
+      <collision>
+        <geometry>
+          <cylinder radius="${wheel_radius}" length="${wheel_width}"/>
+        </geometry>
+      </collision>
+      <inertial>
+        <mass value="0.8"/>
+        <inertia ixx="0.002" ixy="0.0" ixz="0.0"
+                             iyy="0.002" iyz="0.0"
+                                         izz="0.003"/>
+      </inertial>
+    </link>
+  </xacro:macro>
+  <!-- 四個差速輪 -->
+  <xacro:wheel name="front_left_wheel"  x="${ wheel_x}" y="${ wheel_y}"/>
+  <xacro:wheel name="front_right_wheel" x="${ wheel_x}" y="${-wheel_y}"/>
+  <xacro:wheel name="rear_left_wheel"   x="${-wheel_x}" y="${ wheel_y}"/>
+  <xacro:wheel name="rear_right_wheel"  x="${-wheel_x}" y="${-wheel_y}"/>
   <!-- ===== LiDAR link ===== -->
   <joint name="lidar_joint" type="fixed">
@@ -184,11 +115,13 @@
     </sensor>
   </gazebo>
-  <!-- ===== Gazebo diff-drive plugin ===== -->
+  <!-- ===== Gazebo diff-drive plugin（4輪）===== -->
   <gazebo>
     <plugin filename="gz-sim-diff-drive-system"
             name="gz::sim::systems::DiffDrive">
-      <left_joint>left_wheel_joint</left_joint>
-      <right_joint>right_wheel_joint</right_joint>
-      <wheel_separation>${wheel_offset * 2}</wheel_separation>
+      <left_joint>front_left_wheel_joint</left_joint>
+      <left_joint>rear_left_wheel_joint</left_joint>
+      <right_joint>front_right_wheel_joint</right_joint>
+      <right_joint>rear_right_wheel_joint</right_joint>
+      <wheel_separation>${wheel_y * 2}</wheel_separation>
       <wheel_radius>${wheel_radius}</wheel_radius>
       <topic>/cmd_vel</topic>
@@ -198,12 +131,8 @@
     </plugin>
   </gazebo>
-  <!-- Gazebo: zero friction for casters -->
-  <gazebo reference="front_caster">
-    <mu1>0.0</mu1>
-    <mu2>0.0</mu2>
-  </gazebo>
-  <gazebo reference="back_caster">
-    <mu1>0.0</mu1>
-    <mu2>0.0</mu2>
-  </gazebo>
+  <!-- 四輪摩擦力設定 -->
+  <gazebo reference="front_left_wheel">  <mu1>1.0</mu1><mu2>1.0</mu2></gazebo>
+  <gazebo reference="front_right_wheel"> <mu1>1.0</mu1><mu2>1.0</mu2></gazebo>
+  <gazebo reference="rear_left_wheel">   <mu1>1.0</mu1><mu2>1.0</mu2></gazebo>
+  <gazebo reference="rear_right_wheel">  <mu1>1.0</mu1><mu2>1.0</mu2></gazebo>
 </robot>

Commit message: Auto-update: 2026-04-15 17:09

File: src/ammr_bringup/urdf/ammr_base.urdf.xacro (robot description, xacro)
@@ -1,11 +1,10 @@
 <?xml version="1.0"?>
 <robot name="ammr_base" xmlns:xacro="http://www.ros.org/wiki/xacro">
-  <!-- Properties：60cm 直徑圓形底盤 + 4 差速輪 -->
+  <!-- Properties：60cm 直徑圓形底盤 + 4 輪（左右主動差速、前後被動隨動）-->
   <xacro:property name="base_radius"  value="0.30"/>   <!-- 60cm 直徑 -->
   <xacro:property name="base_height"  value="0.12"/>
   <xacro:property name="wheel_radius" value="0.08"/>
   <xacro:property name="wheel_width"  value="0.05"/>
-  <xacro:property name="wheel_x"      value="0.13"/>   <!-- 前後輪距中心距離 -->
-  <xacro:property name="wheel_y"      value="0.24"/>   <!-- 左右輪距中心距離 -->
+  <xacro:property name="wheel_dist"   value="0.26"/>   <!-- 各輪距底盤中心距離 -->
   <!-- base_footprint -->
   <link name="base_footprint"/>
@@ -38,6 +37,6 @@
     </inertial>
   </link>
-  <!-- ===== 輪子 xacro macro ===== -->
-  <xacro:macro name="wheel" params="name x y">
+  <!-- ===== 左/右輪 macro（圓面朝外，軸沿 Y 方向）===== -->
+  <xacro:macro name="lr_wheel" params="name x y">
     <joint name="${name}_joint" type="continuous">
       <parent link="base_link"/>
@@ -68,9 +67,39 @@
     </link>
   </xacro:macro>
-  <!-- 四個差速輪 -->
-  <xacro:wheel name="front_left_wheel"  x="${ wheel_x}" y="${ wheel_y}"/>
-  <xacro:wheel name="front_right_wheel" x="${ wheel_x}" y="${-wheel_y}"/>
-  <xacro:wheel name="rear_left_wheel"   x="${-wheel_x}" y="${ wheel_y}"/>
-  <xacro:wheel name="rear_right_wheel"  x="${-wheel_x}" y="${-wheel_y}"/>
+  <!-- ===== 前/後輪 macro（圓面朝外，軸沿 X 方向）===== -->
+  <xacro:macro name="fb_wheel" params="name x y">
+    <joint name="${name}_joint" type="continuous">
+      <parent link="base_link"/>
+      <child  link="${name}"/>
+      <origin xyz="${x} ${y} ${-base_height/2}" rpy="0 ${pi/2} 0"/>
+      <axis xyz="0 0 1"/>
+    </joint>
+    <link name="${name}">
+      <visual>
+        <geometry>
+          <cylinder radius="${wheel_radius}" length="${wheel_width}"/>
+        </geometry>
+        <material name="dark">
+          <color rgba="0.1 0.1 0.1 1.0"/>
+        </material>
+      </visual>
+      <collision>
+        <geometry>
+          <cylinder radius="${wheel_radius}" length="${wheel_width}"/>
+        </geometry>
+      </collision>
+      <inertial>
+        <mass value="0.8"/>
+        <inertia ixx="0.002" ixy="0.0" ixz="0.0"
+                             iyy="0.002" iyz="0.0"
+                                         izz="0.003"/>
+      </inertial>
+    </link>
+  </xacro:macro>
+  <!-- 四個差速輪（左、右主動；前、後被動）-->
+  <xacro:lr_wheel name="left_wheel"  x="0"              y="${ wheel_dist}"/>
+  <xacro:lr_wheel name="right_wheel" x="0"              y="${-wheel_dist}"/>
+  <xacro:fb_wheel name="front_wheel" x="${ wheel_dist}"  y="0"/>
+  <xacro:fb_wheel name="back_wheel"  x="${-wheel_dist}"  y="0"/>
   <!-- ===== LiDAR link ===== -->
   <joint name="lidar_joint" type="fixed">
@@ -115,13 +144,14 @@
     </sensor>
   </gazebo>
-  <!-- ===== Gazebo diff-drive plugin（4輪）===== -->
+  <!-- ===== Gazebo diff-drive plugin（四輪全驅）===== -->
+  <!-- 左右輪主導差速；前輪歸左組、後輪歸右組，使轉向力矩對稱 -->
   <gazebo>
     <plugin filename="gz-sim-diff-drive-system"
             name="gz::sim::systems::DiffDrive">
-      <left_joint>front_left_wheel_joint</left_joint>
-      <left_joint>rear_left_wheel_joint</left_joint>
-      <right_joint>front_right_wheel_joint</right_joint>
-      <right_joint>rear_right_wheel_joint</right_joint>
-      <wheel_separation>${wheel_y * 2}</wheel_separation>
+      <left_joint>left_wheel_joint</left_joint>
+      <left_joint>front_wheel_joint</left_joint>
+      <right_joint>right_wheel_joint</right_joint>
+      <right_joint>back_wheel_joint</right_joint>
+      <wheel_separation>${wheel_dist * 2}</wheel_separation>
       <wheel_radius>${wheel_radius}</wheel_radius>
       <topic>/cmd_vel</topic>
@@ -132,7 +162,7 @@
   </gazebo>
   <!-- 四輪摩擦力設定 -->
-  <gazebo reference="front_left_wheel">  <mu1>1.0</mu1><mu2>1.0</mu2></gazebo>
-  <gazebo reference="front_right_wheel"> <mu1>1.0</mu1><mu2>1.0</mu2></gazebo>
-  <gazebo reference="rear_left_wheel">   <mu1>1.0</mu1><mu2>1.0</mu2></gazebo>
-  <gazebo reference="rear_right_wheel">  <mu1>1.0</mu1><mu2>1.0</mu2></gazebo>
+  <gazebo reference="left_wheel">  <mu1>1.0</mu1><mu2>1.0</mu2></gazebo>
+  <gazebo reference="right_wheel"> <mu1>1.0</mu1><mu2>1.0</mu2></gazebo>
+  <gazebo reference="front_wheel"> <mu1>1.0</mu1><mu2>1.0</mu2></gazebo>
+  <gazebo reference="back_wheel">  <mu1>1.0</mu1><mu2>1.0</mu2></gazebo>
 </robot>

Commit message: Auto-update: 2026-04-15 18:04

File: src/ammr_bringup/urdf/ammr_base.urdf.xacro (robot description, xacro)
@@ -1,10 +1,11 @@
 <?xml version="1.0"?>
 <robot name="ammr_base" xmlns:xacro="http://www.ros.org/wiki/xacro">
-  <!-- Properties：60cm 直徑圓形底盤 + 4 輪（左右主動差速、前後被動隨動）-->
+  <!-- Properties：60cm 直徑圓形底盤 + 4 全向輪（四角落 mecanum 佈局）-->
   <xacro:property name="base_radius"  value="0.30"/>   <!-- 60cm 直徑 -->
   <xacro:property name="base_height"  value="0.12"/>
   <xacro:property name="wheel_radius" value="0.08"/>
   <xacro:property name="wheel_width"  value="0.05"/>
-  <xacro:property name="wheel_dist"   value="0.26"/>   <!-- 各輪距底盤中心距離 -->
+  <xacro:property name="wheel_x"      value="0.20"/>   <!-- 前後軸距 (m) -->
+  <xacro:property name="wheel_y"      value="0.20"/>   <!-- 左右輪距 (m) -->
   <!-- base_footprint -->
   <link name="base_footprint"/>
@@ -31,5 +32,4 @@
     <inertial>
       <mass value="15.0"/>
-      <!-- 實心圓柱慣性矩 -->
       <inertia ixx="0.356" ixy="0.0" ixz="0.0"
                            iyy="0.356" iyz="0.0"
@@ -37,6 +37,6 @@
     </inertial>
   </link>
-  <!-- ===== 左/右輪 macro（圓面朝外，軸沿 Y 方向）===== -->
-  <xacro:macro name="lr_wheel" params="name x y">
+  <!-- ===== 全向輪 macro（軸沿 Y，四角落）===== -->
+  <xacro:macro name="omni_wheel" params="name x y">
     <joint name="${name}_joint" type="continuous">
       <parent link="base_link"/>
@@ -67,39 +67,9 @@
     </link>
   </xacro:macro>
-  <!-- ===== 前/後輪 macro（圓面朝外，軸沿 X 方向）===== -->
-  <xacro:macro name="fb_wheel" params="name x y">
-    <joint name="${name}_joint" type="continuous">
-      <parent link="base_link"/>
-      <child  link="${name}"/>
-      <origin xyz="${x} ${y} ${-base_height/2}" rpy="0 ${pi/2} 0"/>
-      <axis xyz="0 0 1"/>
-    </joint>
-    <link name="${name}">
-      <visual>
-        <geometry>
-          <cylinder radius="${wheel_radius}" length="${wheel_width}"/>
-        </geometry>
-        <material name="dark">
-          <color rgba="0.1 0.1 0.1 1.0"/>
-        </material>
-      </visual>
-      <collision>
-        <geometry>
-          <cylinder radius="${wheel_radius}" length="${wheel_width}"/>
-        </geometry>
-      </collision>
-      <inertial>
-        <mass value="0.8"/>
-        <inertia ixx="0.002" ixy="0.0" ixz="0.0"
-                             iyy="0.002" iyz="0.0"
-                                         izz="0.003"/>
-      </inertial>
-    </link>
-  </xacro:macro>
-  <!-- 四個差速輪（左、右主動；前、後被動）-->
-  <xacro:lr_wheel name="left_wheel"  x="0"              y="${ wheel_dist}"/>
-  <xacro:lr_wheel name="right_wheel" x="0"              y="${-wheel_dist}"/>
-  <xacro:fb_wheel name="front_wheel" x="${ wheel_dist}"  y="0"/>
-  <xacro:fb_wheel name="back_wheel"  x="${-wheel_dist}"  y="0"/>
+  <!-- 四個全向輪（四角落）-->
+  <xacro:omni_wheel name="front_left_wheel"  x="${ wheel_x}" y="${ wheel_y}"/>
+  <xacro:omni_wheel name="front_right_wheel" x="${ wheel_x}" y="${-wheel_y}"/>
+  <xacro:omni_wheel name="rear_left_wheel"   x="${-wheel_x}" y="${ wheel_y}"/>
+  <xacro:omni_wheel name="rear_right_wheel"  x="${-wheel_x}" y="${-wheel_y}"/>
   <!-- ===== LiDAR link ===== -->
   <joint name="lidar_joint" type="fixed">
@@ -144,14 +114,14 @@
     </sensor>
   </gazebo>
-  <!-- ===== Gazebo diff-drive plugin（四輪全驅）===== -->
-  <!-- 左右輪主導差速；前輪歸左組、後輪歸右組，使轉向力矩對稱 -->
+  <!-- ===== Gazebo Mecanum Drive plugin（全向驅動）===== -->
   <gazebo>
-    <plugin filename="gz-sim-diff-drive-system"
-            name="gz::sim::systems::DiffDrive">
-      <left_joint>left_wheel_joint</left_joint>
-      <left_joint>front_wheel_joint</left_joint>
-      <right_joint>right_wheel_joint</right_joint>
-      <right_joint>back_wheel_joint</right_joint>
-      <wheel_separation>${wheel_dist * 2}</wheel_separation>
+    <plugin filename="gz-sim-mecanum-drive-system"
+            name="gz::sim::systems::MecanumDrive">
+      <front_left_joint>front_left_wheel_joint</front_left_joint>
+      <front_right_joint>front_right_wheel_joint</front_right_joint>
+      <back_left_joint>rear_left_wheel_joint</back_left_joint>
+      <back_right_joint>rear_right_wheel_joint</back_right_joint>
+      <wheel_separation>${wheel_y * 2}</wheel_separation>
+      <wheelbase>${wheel_x * 2}</wheelbase>
       <wheel_radius>${wheel_radius}</wheel_radius>
       <topic>/cmd_vel</topic>
@@ -162,7 +132,7 @@
   </gazebo>
   <!-- 四輪摩擦力設定 -->
-  <gazebo reference="left_wheel">  <mu1>1.0</mu1><mu2>1.0</mu2></gazebo>
-  <gazebo reference="right_wheel"> <mu1>1.0</mu1><mu2>1.0</mu2></gazebo>
-  <gazebo reference="front_wheel"> <mu1>1.0</mu1><mu2>1.0</mu2></gazebo>
-  <gazebo reference="back_wheel">  <mu1>1.0</mu1><mu2>1.0</mu2></gazebo>
+  <gazebo reference="front_left_wheel">  <mu1>1.0</mu1><mu2>1.0</mu2></gazebo>
+  <gazebo reference="front_right_wheel"> <mu1>1.0</mu1><mu2>1.0</mu2></gazebo>
+  <gazebo reference="rear_left_wheel">   <mu1>1.0</mu1><mu2>1.0</mu2></gazebo>
+  <gazebo reference="rear_right_wheel">  <mu1>1.0</mu1><mu2>1.0</mu2></gazebo>
 </robot>
