Commit message: Auto-update: 2026-06-25 15:36

File: src/my_omnibot_description/urdf/omni_bot.urdf.xacro (robot description, xacro)
@@ -37,5 +37,5 @@
       <origin xyz="0 0 0" rpy="0 0 0"/>
       <geometry>
-        <mesh filename="package://my_omnibot_description/meshes/chassis_frame.stl" scale="1 1 1"/>
+        <mesh filename="file://$(find my_omnibot_description)/meshes/chassis_frame.stl" scale="1 1 1"/>
       </geometry>
       <material name="chassis_gray"><color rgba="0.55 0.55 0.58 1.0"/></material>

File: src/my_omnibot_description/urdf/roller.xacro (robot description, xacro)
@@ -18,5 +18,5 @@
       <visual>
         <geometry>
-          <mesh filename="package://my_omnibot_description/meshes/roller_omni_wheel.stl" scale="1 1 1"/>
+          <mesh filename="file://$(find my_omnibot_description)/meshes/roller_omni_wheel.stl" scale="1 1 1"/>
         </geometry>
       </visual>

Commit message: Auto-update: 2026-06-25 15:45

File: src/my_omnibot_description/urdf/omni_bot.urdf.xacro (robot description, xacro)
@@ -39,5 +39,5 @@
         <mesh filename="file://$(find my_omnibot_description)/meshes/chassis_frame.stl" scale="1 1 1"/>
       </geometry>
-      <material name="chassis_gray"><color rgba="0.55 0.55 0.58 1.0"/></material>
+      <material name="chassis_orange"><color rgba="0.95 0.45 0.10 1.0"/></material>
     </visual>
     <collision>

Commit message: Auto-update: 2026-06-25 15:51

File: src/my_omnibot_description/urdf/omni_bot.urdf.xacro (robot description, xacro)
@@ -39,5 +39,5 @@
         <mesh filename="file://$(find my_omnibot_description)/meshes/chassis_frame.stl" scale="1 1 1"/>
       </geometry>
-      <material name="chassis_orange"><color rgba="0.95 0.45 0.10 1.0"/></material>
+      <material name="chassis_blue"><color rgba="0.15 0.45 0.85 1.0"/></material>
     </visual>
     <collision>
