Commit message: Auto-update: 2026-07-28 04:11

File: src/my_omnibot_description/urdf/omni_bot.urdf.xacro (robot description, xacro)
@@ -2,4 +2,9 @@
 <robot name="omni_bot" xmlns:xacro="http://www.ros.org/wiki/xacro">
   <xacro:arg name="use_camera" default="true"/>
+  <!-- Phase 2: UFACTORY Lite 6 arm on a mast above the LiDAR. Default OFF so
+       every existing navigation launch/benchmark keeps the exact validated
+       robot; turn on with  use_arm:=true . -->
+  <xacro:arg name="use_arm" default="false"/>
+  <xacro:arg name="arm_ros2_control_plugin" default="gz_ros2_control/GazeboSimSystem"/>
   <xacro:include filename="$(find my_omnibot_description)/urdf/rim.xacro"/>
   <xacro:include filename="$(find my_omnibot_description)/urdf/lidar.xacro"/>
@@ -108,3 +113,41 @@
     </plugin>
   </gazebo>
+  <!-- ===== Phase 2: manipulator (UFACTORY Lite 6, 6-DOF) ================
+       Mounted on a mast ABOVE the LiDAR (see arm_mount.xacro for why).
+       Base 3 DOF (x, y, theta) + arm 6 DOF = 9 DOF against a 6-DOF SE(3)
+       end-effector task -> 3 redundant DOF for whole-body coordination.
+       ===================================================================== -->
+  <xacro:if value="$(arg use_arm)">
+    <xacro:include filename="$(find my_omnibot_description)/urdf/arm_mount.xacro"/>
+    <!-- xarm_description expects these three globals. Upstream sets them in
+         _private_macro.xacro with scope="parent", which only works when that
+         file is pulled in from INSIDE a macro; included at robot level it
+         raises "'dict' object has no attribute '_setitem'". Declaring them
+         here directly is equivalent. -->
+    <xacro:property name="is_ros2" value="true"/>
+    <xacro:property name="use_xacro_load_yaml" value="true"/>
+    <xacro:property name="use_len" value="true"/>
+    <!-- shared link/material/gazebo helpers the lite6 macros call into
+         (upstream pulls these in from xarm_device_macro.xacro) -->
+    <xacro:include filename="$(find xarm_description)/urdf/common/common.material.xacro"/>
+    <xacro:common_material prefix=""/>
+    <!-- Absolute file:// path, because gz Harmonic cannot resolve package://
+         (the same fix the omni_bot chassis and roller meshes needed). -->
+    <xacro:property name="mesh_path" value="file://$(find xarm_description)/meshes"/>
+    <xacro:property name="mesh_suffix" value="stl"/>
+    <xacro:include filename="$(find xarm_description)/urdf/common/common.link.xacro"/>
+    <xacro:include filename="$(find xarm_description)/urdf/common/common.gazebo.xacro"/>
+    <xacro:include filename="$(find xarm_description)/urdf/lite6/lite6_robot_macro.xacro"/>
+    <xacro:arm_mount parent="base_link"/>
+    <xacro:lite6_robot
+      prefix=""
+      ros2_control_plugin="$(arg arm_ros2_control_plugin)"
+      kinematics_params_filename="$(find xarm_description)/config/kinematics/default/lite6_default_kinematics.yaml"/>
+    <!-- arm base bolted to the top of the mast plate -->
+    <joint name="arm_base_joint" type="fixed">
+      <parent link="arm_mount_link"/>
+      <child link="link_base"/>
+      <origin xyz="0 0 0.006" rpy="0 0 0"/>
+    </joint>
+  </xacro:if>
 </robot>

Commit message: Auto-update: 2026-07-28 04:27

File: src/my_omnibot_description/urdf/omni_bot.urdf.xacro (robot description, xacro)
@@ -125,5 +125,9 @@
          raises "'dict' object has no attribute '_setitem'". Declaring them
          here directly is equivalent. -->
-    <xacro:property name="is_ros2" value="true"/>
+    <!-- is_ros2=false makes lite6_robot SKIP its own ros2_control block; we
+         supply lite6_ros2_control_gz.xacro instead, which is identical except
+         that it sets initial_value on the position state interfaces so the arm
+         spawns already tucked instead of at all-zeros. -->
+    <xacro:property name="is_ros2" value="false"/>
     <xacro:property name="use_xacro_load_yaml" value="true"/>
     <xacro:property name="use_len" value="true"/>
@@ -144,4 +148,7 @@
       ros2_control_plugin="$(arg arm_ros2_control_plugin)"
       kinematics_params_filename="$(find xarm_description)/config/kinematics/default/lite6_default_kinematics.yaml"/>
+    <xacro:include filename="$(find my_omnibot_description)/urdf/lite6_ros2_control_gz.xacro"/>
+    <xacro:lite6_ros2_control_gz prefix=""
+      ros2_control_plugin="$(arg arm_ros2_control_plugin)"/>
     <!-- arm base bolted to the top of the mast plate -->
     <joint name="arm_base_joint" type="fixed">

Commit message: Auto-update: 2026-08-04 09:23

File: src/my_omnibot_description/urdf/omni_bot.urdf.xacro (robot description, xacro)
@@ -48,6 +48,18 @@
     <collision>
       <origin xyz="0 0 0.14" rpy="0 0 0"/>
+      <!-- The chassis is a DISC of radius 0.300 m: that is what the visual mesh
+           measures (chassis_frame.stl reaches 0.300 in every 30 deg sector) and
+           it is what the analysis uses to judge clearance. The collision body
+           used to be a 0.45 x 0.45 box, half-extent 0.225, so the simulated
+           robot was 7.5 cm smaller than the real one along its axes, and a
+           reported contact shallower than 7.5 cm had not physically happened in
+           gz at all. Over ~230 trials of the final configuration, 15 events
+           were reported as contacts but only 4 were deeper than that gap, so
+           the two measures disagreed about 11 of them.
+           Note this makes the robot LARGER on its axes (0.300 vs 0.225) and
+           slightly smaller on its diagonals (0.300 vs 0.225*sqrt(2) = 0.318),
+           so earlier batches are not comparable to anything run after it. -->
       <geometry>
-        <box size="0.45 0.45 0.18"/>
+        <cylinder radius="0.300" length="0.18"/>
       </geometry>
     </collision>

Commit message: Auto-update: 2026-08-26 17:47

File: src/my_omnibot_description/urdf/omni_bot.urdf.xacro (robot description, xacro)
@@ -6,6 +6,9 @@
        robot; turn on with  use_arm:=true . -->
   <xacro:arg name="use_arm" default="false"/>
+  <!-- Factory gripper on the arm. Default false: it adds a commanded joint and
+       a mimic joint, and every existing navigation benchmark must keep running
+       the exact robot it was validated on. -->
+  <xacro:arg name="add_gripper" default="false"/>
   <xacro:arg name="arm_ros2_control_plugin" default="gz_ros2_control/GazeboSimSystem"/>
-  <xacro:include filename="$(find my_omnibot_description)/urdf/rim.xacro"/>
   <xacro:include filename="$(find my_omnibot_description)/urdf/lidar.xacro"/>
   <!-- ===================================================================
@@ -32,42 +35,8 @@
     <origin xyz="0 0 ${wheel_r}" rpy="0 0 0"/>
   </joint>
-  <!-- Chassis body (visual = original mesh, collision = simple raised box) -->
-  <link name="base_link">
-    <inertial>
-      <origin xyz="0 0 0.14" rpy="0 0 0"/>
-      <mass value="18.0"/>
-      <inertia ixx="0.5229" ixy="0.0" ixz="0.0" iyy="0.5229" iyz="0.0" izz="0.81"/>
-    </inertial>
-    <visual>
-      <origin xyz="0 0 0" rpy="0 0 0"/>
-      <geometry>
-        <mesh filename="file://$(find my_omnibot_description)/meshes/chassis_frame.stl" scale="1 1 1"/>
-      </geometry>
-      <material name="chassis_blue"><color rgba="0.15 0.45 0.85 1.0"/></material>
-    </visual>
-    <collision>
-      <origin xyz="0 0 0.14" rpy="0 0 0"/>
-      <!-- The chassis is a DISC of radius 0.300 m: that is what the visual mesh
-           measures (chassis_frame.stl reaches 0.300 in every 30 deg sector) and
-           it is what the analysis uses to judge clearance. The collision body
-           used to be a 0.45 x 0.45 box, half-extent 0.225, so the simulated
-           robot was 7.5 cm smaller than the real one along its axes, and a
-           reported contact shallower than 7.5 cm had not physically happened in
-           gz at all. Over ~230 trials of the final configuration, 15 events
-           were reported as contacts but only 4 were deeper than that gap, so
-           the two measures disagreed about 11 of them.
-           Note this makes the robot LARGER on its axes (0.300 vs 0.225) and
-           slightly smaller on its diagonals (0.300 vs 0.225*sqrt(2) = 0.318),
-           so earlier batches are not comparable to anything run after it. -->
-      <geometry>
-        <cylinder radius="0.300" length="0.18"/>
-      </geometry>
-    </collision>
-  </link>
-  <!-- ===== Omni wheels (visual decoration) ===== -->
-  <xacro:rim name="a" parent="base_link" xyz="0.245 0 0"  rpy="0 -1.57 0"  color="0.2 0.7 0.2 1"/>
-  <xacro:rim name="b" parent="base_link" xyz="0 0.245 0"  rpy="1.57 1.57 0" color="0.2 0.4 0.8 1"/>
-  <xacro:rim name="c" parent="base_link" xyz="-0.245 0 0" rpy="0 1.57 0"   color="0.85 0.75 0.2 1"/>
-  <xacro:rim name="d" parent="base_link" xyz="0 -0.245 0" rpy="-1.57 -1.57 0" color="0.8 0.2 0.2 1"/>
+  <!-- Chassis body + the four omni wheels. Extracted to chassis_body.xacro so
+       the whole-body kinematics model uses the same geometry; see that file. -->
+  <xacro:include filename="$(find my_omnibot_description)/urdf/chassis_body.xacro"/>
+  <xacro:chassis_body/>
   <!-- ===== Hidden zero-friction support wheels (collision only) ===== -->
   <xacro:macro name="support" params="name x y">
@@ -162,5 +131,22 @@
     <xacro:include filename="$(find my_omnibot_description)/urdf/lite6_ros2_control_gz.xacro"/>
     <xacro:lite6_ros2_control_gz prefix=""
-      ros2_control_plugin="$(arg arm_ros2_control_plugin)"/>
+      ros2_control_plugin="$(arg arm_ros2_control_plugin)"
+      add_gripper="$(arg add_gripper)"/>
+    <!-- Factory gripper. link_eef has to be declared here: upstream puts it in
+         xarm_device_macro.xacro, which we do not include, and lite6.urdf.xacro
+         has its copy commented out. Only the URDF half of the gripper is
+         pulled in; the full uflite_gripper_macro also drags in its own
+         ros2_control system, transmissions and a gazebo grasp-fix plugin, and
+         the finger joint is already declared in our single ros2_control block. -->
+    <xacro:if value="$(arg add_gripper)">
+      <link name="link_eef"/>
+      <joint name="joint_eef" type="fixed">
+        <parent link="link6"/>
+        <child link="link_eef"/>
+        <origin xyz="0 0 0" rpy="0 0 0"/>
+      </joint>
+      <xacro:include filename="$(find xarm_description)/urdf/gripper/uflite_gripper.urdf.xacro"/>
+      <xacro:uflite_gripper_urdf prefix="" attach_to="link_eef"/>
+    </xacro:if>
     <!-- arm base bolted to the top of the mast plate -->
     <joint name="arm_base_joint" type="fixed">
@@ -169,4 +155,11 @@
       <origin xyz="0 0 0.006" rpy="0 0 0"/>
     </joint>
+    <!-- Observation frames for arm avoidance. Massless and geometry-free, so
+         gz lumps them into the parent link and physics is unchanged; they exist
+         only so robot_state_publisher puts them on TF for
+         ammr_wholebody_mpc/arm_detection_points.py. Shared with
+         omni_bot_wholebody.urdf.xacro so both models agree by construction. -->
+    <xacro:include filename="$(find my_omnibot_description)/urdf/arm_detect_points.xacro"/>
+    <xacro:arm_detect_points/>
     <!-- runs a controller_manager inside gz so the 6 arm joints are simulated
          at the physics rate. The base keeps using gz VelocityControl on

Commit message: Auto-update: 2026-08-26 18:21

File: src/my_omnibot_description/urdf/omni_bot.urdf.xacro (robot description, xacro)
@@ -95,10 +95,9 @@
   </gazebo>
   <!-- ===== Phase 2: manipulator (UFACTORY Lite 6, 6-DOF) ================
-       Mounted on a mast ABOVE the LiDAR (see arm_mount.xacro for why).
+       Attached at the real robot's mounting point, base_link + (0.11, 0, 0.28).
        Base 3 DOF (x, y, theta) + arm 6 DOF = 9 DOF against a 6-DOF SE(3)
        end-effector task -> 3 redundant DOF for whole-body coordination.
        ===================================================================== -->
   <xacro:if value="$(arg use_arm)">
-    <xacro:include filename="$(find my_omnibot_description)/urdf/arm_mount.xacro"/>
     <!-- xarm_description expects these three globals. Upstream sets them in
          _private_macro.xacro with scope="parent", which only works when that
@@ -124,5 +123,4 @@
     <xacro:include filename="$(find xarm_description)/urdf/common/common.gazebo.xacro"/>
     <xacro:include filename="$(find xarm_description)/urdf/lite6/lite6_robot_macro.xacro"/>
-    <xacro:arm_mount parent="base_link"/>
     <xacro:lite6_robot
       prefix=""
@@ -149,9 +147,18 @@
       <xacro:uflite_gripper_urdf prefix="" attach_to="link_eef"/>
     </xacro:if>
-    <!-- arm base bolted to the top of the mast plate -->
+    <!-- Arm attach point, verbatim from the real robot: base_link + (0.11, 0,
+         0.28). Same values as mobile_manipulator.xacro (attach_xyz default) and
+         fake_mobile_manipulator_modified.urdf (base_link_to_link_base) in the
+         MastersThesis_ros tree.
+         No mount structure is modelled, matching that reference, which bolts
+         the arm straight to base_link. An earlier version of this file put the
+         arm on a centred mast whose risers hid in the LiDAR sectors scan_relay
+         already masks; that geometry does not survive the 0.11 m offset (the
+         masked sectors stop intersecting the plate footprint), and the real
+         bracket is not measured, so nothing is invented in its place. -->
     <joint name="arm_base_joint" type="fixed">
-      <parent link="arm_mount_link"/>
+      <parent link="base_link"/>
       <child link="link_base"/>
-      <origin xyz="0 0 0.006" rpy="0 0 0"/>
+      <origin xyz="0.11 0 0.28" rpy="0 0 0"/>
     </joint>
     <!-- Observation frames for arm avoidance. Massless and geometry-free, so

File: src/my_omnibot_description/urdf/omni_bot_wholebody.urdf.xacro (robot description, xacro)
@@ -10,5 +10,5 @@
             [base_theta revolute  Z] -> base_theta_link
             [fixed, z + 0.05]        -> base_link
-            [arm_mount + fixed]      -> link_base -> joint1..6 -> link_eef
+            [fixed, 0.11 0 0.28]     -> link_base -> joint1..6 -> link_eef
   so a standard kinematics library (KDL, Pinocchio, MoveIt) sees a 9-DOF arm
   and gives the whole-body Jacobian directly, with no hand-written base/arm
@@ -104,11 +104,7 @@
   <xacro:chassis_body/>
   <!-- ================= arm, on the real mount ===================== -->
-  <!-- The ROS 1 model bolted the arm straight to base_link at 0.11 0 0.28.
-       We keep our own mount instead: centred, on a mast whose risers sit in
-       the LiDAR sectors scan_relay already masks. Using a different attach
-       point here than in simulation would make the solver plan for a robot
-       that does not exist, so this MUST stay in step with omni_bot.urdf.xacro. -->
-  <xacro:include filename="$(find my_omnibot_description)/urdf/arm_mount.xacro"/>
-  <xacro:arm_mount parent="base_link"/>
+  <!-- The attach point MUST stay in step with omni_bot.urdf.xacro: a solver
+       that placed the arm somewhere the simulator does not would plan for a
+       robot that has never been run. -->
   <xacro:property name="is_ros2" value="false"/>
   <xacro:property name="use_xacro_load_yaml" value="true"/>
@@ -125,8 +121,18 @@
     ros2_control_plugin=""
     kinematics_params_filename="$(find xarm_description)/config/kinematics/default/lite6_default_kinematics.yaml"/>
+  <!-- Arm attach point, verbatim from the real robot: base_link + (0.11, 0,
+       0.28). Same values as mobile_manipulator.xacro (attach_xyz default) and
+       fake_mobile_manipulator_modified.urdf (base_link_to_link_base) in the
+       MastersThesis_ros tree.
+       No mount structure is modelled, matching that reference, which bolts
+       the arm straight to base_link. An earlier version of this file put the
+       arm on a centred mast whose risers hid in the LiDAR sectors scan_relay
+       already masks; that geometry does not survive the 0.11 m offset (the
+       masked sectors stop intersecting the plate footprint), and the real
+       bracket is not measured, so nothing is invented in its place. -->
   <joint name="arm_base_joint" type="fixed">
-    <parent link="arm_mount_link"/>
+    <parent link="base_link"/>
     <child link="link_base"/>
-    <origin xyz="0 0 0.006" rpy="0 0 0"/>
+    <origin xyz="0.11 0 0.28" rpy="0 0 0"/>
   </joint>
   <!-- ================= factory gripper + TCP ====================== -->
