Commit message: Auto-update: 2026-07-28 04:50

File: src/my_omnibot_description/urdf/lite6_ros2_control_gz.xacro (robot description, xacro)
@@ -10,23 +10,25 @@
   <param name="initial_value"> on the position state interface, so declaring the
   block here lets the robot spawn already tucked.
-  TUCK pose (found by searching the joint space with FK, see the reasoning in
-  the progress notes):
-      joint2 -2.418, joint3 +4.953, joint5 -1.964, rest 0
-  It satisfies, simultaneously:
-      * every link origin stays >= 0.40 m, i.e. >0.12 m above the chassis top
-        (0.28 m) so the arm never rests on the base,
-      * horizontal radius 0.133 m, well inside the 0.30 m base radius, so the
-        arm does not stick out past the footprint the costmap plans with,
-      * >= 0.20 rad away from every joint limit, so the controller is not
-        starting against a hard stop.
-  Compare with all-zeros: radius 0.087 m but z 0.490..0.780, i.e. the arm stands
-  tall and folds back over itself.
+  TUCK pose, chosen with the real collision meshes (not just joint frames):
+      joint2 -0.082, joint3 +0.089, joint5 +1.679, rest 0
+  The problem it fixes: at the official all-zeros "home" the wrist (link6) bottoms
+  out at z = 0.490 while the arm's own base housing (link_base) tops out at
+  0.509, so the hand hangs 2 cm BELOW the base and reads as "inside" the mount.
+  Rotating joint5 lifts the wrist clear.
+  Verified with src/my_omnibot_description/scripts/find_tuck_pose.py:
+      lowest moving link  0.527 m  (+0.018 above the arm base top)
+      horizontal radius   0.155 m  (inside the 0.30 m chassis radius, so the
+                                    costmap footprint used for navigation still
+                                    covers the arm)
+      highest point       0.828 m
+  All-zeros for comparison: 0.490 / 0.143 / 0.820, i.e. the same envelope but
+  dipping below the base.
 -->
 <robot xmlns:xacro="http://www.ros.org/wiki/xacro">
   <xacro:property name="tuck_j1" value="0.0"/>
-  <xacro:property name="tuck_j2" value="-2.418"/>
-  <xacro:property name="tuck_j3" value="4.953"/>
+  <xacro:property name="tuck_j2" value="-0.082"/>
+  <xacro:property name="tuck_j3" value="0.089"/>
   <xacro:property name="tuck_j4" value="0.0"/>
-  <xacro:property name="tuck_j5" value="-1.964"/>
+  <xacro:property name="tuck_j5" value="1.679"/>
   <xacro:property name="tuck_j6" value="0.0"/>
   <xacro:macro name="lite6_ros2_control_gz"

Commit message: Auto-update: 2026-08-26 17:35

File: src/my_omnibot_description/urdf/lite6_ros2_control_gz.xacro (robot description, xacro)
@@ -33,5 +33,6 @@
   <xacro:property name="tuck_j6" value="0.0"/>
   <xacro:macro name="lite6_ros2_control_gz"
-               params="prefix:='' ros2_control_plugin:='gz_ros2_control/GazeboSimSystem'">
+               params="prefix:='' ros2_control_plugin:='gz_ros2_control/GazeboSimSystem'
+                       add_gripper:=false">
     <ros2_control name="${prefix}lite6_gz" type="system">
       <hardware>
@@ -61,4 +62,25 @@
       <xacro:arm_joint num="5" lower="-2.1642"     upper="2.1642"     initial="${tuck_j5}"/>
       <xacro:arm_joint num="6" lower="${-2.0*pi}"  upper="${2.0*pi}"  initial="${tuck_j6}"/>
+      <!-- UFACTORY Lite 6 factory gripper. Only finger_joint1 is commanded:
+           finger_joint2 carries a <mimic> tag in uflite_gripper.urdf.xacro and
+           gz_ros2_control follows it from the URDF, so declaring it here as
+           well would give two writers for one joint.
+           Upstream's uflite_gripper.ros2_control.xacro is not reused because it
+           opens a SECOND <ros2_control> system. Two systems means two hardware
+           components in one gz world, and the arm and the gripper then come up
+           independently: the gripper can be live while the arm is not. One
+           system keeps them in step. -->
+      <xacro:if value="${add_gripper}">
+        <joint name="${prefix}finger_joint1">
+          <command_interface name="position">
+            <param name="min">0.0</param>
+            <param name="max">0.0089</param>
+          </command_interface>
+          <state_interface name="position">
+            <param name="initial_value">0.0</param>
+          </state_interface>
+          <state_interface name="velocity"/>
+        </joint>
+      </xacro:if>
     </ros2_control>
   </xacro:macro>

File: src/my_omnibot_description/urdf/omni_bot.urdf.xacro (robot description, xacro)
@@ -6,6 +6,9 @@
        robot; turn on with  use_arm:=true . -->
   <xacro:arg name="use_arm" default="false"/>
+  <!-- Factory gripper on the arm. Default false: it adds a commanded joint and
+       a mimic joint, and every existing navigation benchmark must keep running
+       the exact robot it was validated on. -->
+  <xacro:arg name="add_gripper" default="false"/>
   <xacro:arg name="arm_ros2_control_plugin" default="gz_ros2_control/GazeboSimSystem"/>
-  <xacro:include filename="$(find my_omnibot_description)/urdf/rim.xacro"/>
   <xacro:include filename="$(find my_omnibot_description)/urdf/lidar.xacro"/>
   <!-- ===================================================================
@@ -32,42 +35,8 @@
     <origin xyz="0 0 ${wheel_r}" rpy="0 0 0"/>
   </joint>
-  <!-- Chassis body (visual = original mesh, collision = simple raised box) -->
-  <link name="base_link">
-    <inertial>
-      <origin xyz="0 0 0.14" rpy="0 0 0"/>
-      <mass value="18.0"/>
-      <inertia ixx="0.5229" ixy="0.0" ixz="0.0" iyy="0.5229" iyz="0.0" izz="0.81"/>
-    </inertial>
-    <visual>
-      <origin xyz="0 0 0" rpy="0 0 0"/>
-      <geometry>
-        <mesh filename="file://$(find my_omnibot_description)/meshes/chassis_frame.stl" scale="1 1 1"/>
-      </geometry>
-      <material name="chassis_blue"><color rgba="0.15 0.45 0.85 1.0"/></material>
-    </visual>
-    <collision>
-      <origin xyz="0 0 0.14" rpy="0 0 0"/>
-      <!-- The chassis is a DISC of radius 0.300 m: that is what the visual mesh
-           measures (chassis_frame.stl reaches 0.300 in every 30 deg sector) and
-           it is what the analysis uses to judge clearance. The collision body
-           used to be a 0.45 x 0.45 box, half-extent 0.225, so the simulated
-           robot was 7.5 cm smaller than the real one along its axes, and a
-           reported contact shallower than 7.5 cm had not physically happened in
-           gz at all. Over ~230 trials of the final configuration, 15 events
-           were reported as contacts but only 4 were deeper than that gap, so
-           the two measures disagreed about 11 of them.
-           Note this makes the robot LARGER on its axes (0.300 vs 0.225) and
-           slightly smaller on its diagonals (0.300 vs 0.225*sqrt(2) = 0.318),
-           so earlier batches are not comparable to anything run after it. -->
-      <geometry>
-        <cylinder radius="0.300" length="0.18"/>
-      </geometry>
-    </collision>
-  </link>
-  <!-- ===== Omni wheels (visual decoration) ===== -->
-  <xacro:rim name="a" parent="base_link" xyz="0.245 0 0"  rpy="0 -1.57 0"  color="0.2 0.7 0.2 1"/>
-  <xacro:rim name="b" parent="base_link" xyz="0 0.245 0"  rpy="1.57 1.57 0" color="0.2 0.4 0.8 1"/>
-  <xacro:rim name="c" parent="base_link" xyz="-0.245 0 0" rpy="0 1.57 0"   color="0.85 0.75 0.2 1"/>
-  <xacro:rim name="d" parent="base_link" xyz="0 -0.245 0" rpy="-1.57 -1.57 0" color="0.8 0.2 0.2 1"/>
+  <!-- Chassis body + the four omni wheels. Extracted to chassis_body.xacro so
+       the whole-body kinematics model uses the same geometry; see that file. -->
+  <xacro:include filename="$(find my_omnibot_description)/urdf/chassis_body.xacro"/>
+  <xacro:chassis_body/>
   <!-- ===== Hidden zero-friction support wheels (collision only) ===== -->
   <xacro:macro name="support" params="name x y">
@@ -162,5 +131,22 @@
     <xacro:include filename="$(find my_omnibot_description)/urdf/lite6_ros2_control_gz.xacro"/>
     <xacro:lite6_ros2_control_gz prefix=""
-      ros2_control_plugin="$(arg arm_ros2_control_plugin)"/>
+      ros2_control_plugin="$(arg arm_ros2_control_plugin)"
+      add_gripper="$(arg add_gripper)"/>
+    <!-- Factory gripper. link_eef has to be declared here: upstream puts it in
+         xarm_device_macro.xacro, which we do not include, and lite6.urdf.xacro
+         has its copy commented out. Only the URDF half of the gripper is
+         pulled in; the full uflite_gripper_macro also drags in its own
+         ros2_control system, transmissions and a gazebo grasp-fix plugin, and
+         the finger joint is already declared in our single ros2_control block. -->
+    <xacro:if value="$(arg add_gripper)">
+      <link name="link_eef"/>
+      <joint name="joint_eef" type="fixed">
+        <parent link="link6"/>
+        <child link="link_eef"/>
+        <origin xyz="0 0 0" rpy="0 0 0"/>
+      </joint>
+      <xacro:include filename="$(find xarm_description)/urdf/gripper/uflite_gripper.urdf.xacro"/>
+      <xacro:uflite_gripper_urdf prefix="" attach_to="link_eef"/>
+    </xacro:if>
     <!-- arm base bolted to the top of the mast plate -->
     <joint name="arm_base_joint" type="fixed">

File: src/my_omnibot_description/urdf/omni_bot_wholebody.urdf.xacro (robot description, xacro)
@@ -15,8 +15,11 @@
   composition. That is the entire reason this file exists, and it is what makes
   base and arm solvable in one QP rather than two stacked controllers.
-  NOT a simulation model. Every link is massless, there are no wheels, no
-  rollers, no sensors and no gz plugins. gz keeps using omni_bot.urdf.xacro;
-  this one is for the solver only. The ROS 1 file called itself "fake" for the
-  same reason.
+  NOT a simulation model: no sensors, no gz plugins, no controllers, and the
+  three virtual base links carry only token inertia. It does carry the real
+  chassis and wheels, because the solver has to know what the arm can hit and
+  because a model without them is not recognisable in Foxglove. gz keeps using
+  omni_bot.urdf.xacro; this one is for the solver only. The ROS 1 file called
+  itself "fake" for the same reason, and it went further, dropping the wheels
+  as well.
   Two numbers deliberately differ from the ROS 1 original:
     base_x / base_y velocity   the original allowed 0.3 m/s per axis. Our
@@ -93,5 +96,11 @@
     <origin xyz="0 0 0.05" rpy="0 0 0"/>
   </joint>
-  <xacro:ghost_link name="base_link"/>
+  <!-- The real chassis: mesh visual, the 0.300 m collision cylinder every
+       clearance number is measured against, and the four omni wheels. Shared
+       with the simulation model, so the solver checks the arm against the same
+       body gz simulates. Without it the arm could plan straight through its own
+       base and the model would look like a floating arm in Foxglove. -->
+  <xacro:include filename="$(find my_omnibot_description)/urdf/chassis_body.xacro"/>
+  <xacro:chassis_body/>
   <!-- ================= arm, on the real mount ===================== -->
   <!-- The ROS 1 model bolted the arm straight to base_link at 0.11 0 0.28.

Commit message: Auto-update: 2026-08-26 17:40

File: src/my_omnibot_description/urdf/lite6_ros2_control_gz.xacro (robot description, xacro)
@@ -33,6 +33,5 @@
   <xacro:property name="tuck_j6" value="0.0"/>
   <xacro:macro name="lite6_ros2_control_gz"
-               params="prefix:='' ros2_control_plugin:='gz_ros2_control/GazeboSimSystem'
-                       add_gripper:=false">
+               params="prefix:='' ros2_control_plugin:='gz_ros2_control/GazeboSimSystem'">
     <ros2_control name="${prefix}lite6_gz" type="system">
       <hardware>
@@ -62,25 +61,4 @@
       <xacro:arm_joint num="5" lower="-2.1642"     upper="2.1642"     initial="${tuck_j5}"/>
       <xacro:arm_joint num="6" lower="${-2.0*pi}"  upper="${2.0*pi}"  initial="${tuck_j6}"/>
-      <!-- UFACTORY Lite 6 factory gripper. Only finger_joint1 is commanded:
-           finger_joint2 carries a <mimic> tag in uflite_gripper.urdf.xacro and
-           gz_ros2_control follows it from the URDF, so declaring it here as
-           well would give two writers for one joint.
-           Upstream's uflite_gripper.ros2_control.xacro is not reused because it
-           opens a SECOND <ros2_control> system. Two systems means two hardware
-           components in one gz world, and the arm and the gripper then come up
-           independently: the gripper can be live while the arm is not. One
-           system keeps them in step. -->
-      <xacro:if value="${add_gripper}">
-        <joint name="${prefix}finger_joint1">
-          <command_interface name="position">
-            <param name="min">0.0</param>
-            <param name="max">0.0089</param>
-          </command_interface>
-          <state_interface name="position">
-            <param name="initial_value">0.0</param>
-          </state_interface>
-          <state_interface name="velocity"/>
-        </joint>
-      </xacro:if>
     </ros2_control>
   </xacro:macro>

File: src/my_omnibot_description/urdf/omni_bot.urdf.xacro (robot description, xacro)
@@ -6,9 +6,6 @@
        robot; turn on with  use_arm:=true . -->
   <xacro:arg name="use_arm" default="false"/>
-  <!-- Factory gripper on the arm. Default false: it adds a commanded joint and
-       a mimic joint, and every existing navigation benchmark must keep running
-       the exact robot it was validated on. -->
-  <xacro:arg name="add_gripper" default="false"/>
   <xacro:arg name="arm_ros2_control_plugin" default="gz_ros2_control/GazeboSimSystem"/>
+  <xacro:include filename="$(find my_omnibot_description)/urdf/rim.xacro"/>
   <xacro:include filename="$(find my_omnibot_description)/urdf/lidar.xacro"/>
   <!-- ===================================================================
@@ -35,8 +32,42 @@
     <origin xyz="0 0 ${wheel_r}" rpy="0 0 0"/>
   </joint>
-  <!-- Chassis body + the four omni wheels. Extracted to chassis_body.xacro so
-       the whole-body kinematics model uses the same geometry; see that file. -->
-  <xacro:include filename="$(find my_omnibot_description)/urdf/chassis_body.xacro"/>
-  <xacro:chassis_body/>
+  <!-- Chassis body (visual = original mesh, collision = simple raised box) -->
+  <link name="base_link">
+    <inertial>
+      <origin xyz="0 0 0.14" rpy="0 0 0"/>
+      <mass value="18.0"/>
+      <inertia ixx="0.5229" ixy="0.0" ixz="0.0" iyy="0.5229" iyz="0.0" izz="0.81"/>
+    </inertial>
+    <visual>
+      <origin xyz="0 0 0" rpy="0 0 0"/>
+      <geometry>
+        <mesh filename="file://$(find my_omnibot_description)/meshes/chassis_frame.stl" scale="1 1 1"/>
+      </geometry>
+      <material name="chassis_blue"><color rgba="0.15 0.45 0.85 1.0"/></material>
+    </visual>
+    <collision>
+      <origin xyz="0 0 0.14" rpy="0 0 0"/>
+      <!-- The chassis is a DISC of radius 0.300 m: that is what the visual mesh
+           measures (chassis_frame.stl reaches 0.300 in every 30 deg sector) and
+           it is what the analysis uses to judge clearance. The collision body
+           used to be a 0.45 x 0.45 box, half-extent 0.225, so the simulated
+           robot was 7.5 cm smaller than the real one along its axes, and a
+           reported contact shallower than 7.5 cm had not physically happened in
+           gz at all. Over ~230 trials of the final configuration, 15 events
+           were reported as contacts but only 4 were deeper than that gap, so
+           the two measures disagreed about 11 of them.
+           Note this makes the robot LARGER on its axes (0.300 vs 0.225) and
+           slightly smaller on its diagonals (0.300 vs 0.225*sqrt(2) = 0.318),
+           so earlier batches are not comparable to anything run after it. -->
+      <geometry>
+        <cylinder radius="0.300" length="0.18"/>
+      </geometry>
+    </collision>
+  </link>
+  <!-- ===== Omni wheels (visual decoration) ===== -->
+  <xacro:rim name="a" parent="base_link" xyz="0.245 0 0"  rpy="0 -1.57 0"  color="0.2 0.7 0.2 1"/>
+  <xacro:rim name="b" parent="base_link" xyz="0 0.245 0"  rpy="1.57 1.57 0" color="0.2 0.4 0.8 1"/>
+  <xacro:rim name="c" parent="base_link" xyz="-0.245 0 0" rpy="0 1.57 0"   color="0.85 0.75 0.2 1"/>
+  <xacro:rim name="d" parent="base_link" xyz="0 -0.245 0" rpy="-1.57 -1.57 0" color="0.8 0.2 0.2 1"/>
   <!-- ===== Hidden zero-friction support wheels (collision only) ===== -->
   <xacro:macro name="support" params="name x y">
@@ -131,22 +162,5 @@
     <xacro:include filename="$(find my_omnibot_description)/urdf/lite6_ros2_control_gz.xacro"/>
     <xacro:lite6_ros2_control_gz prefix=""
-      ros2_control_plugin="$(arg arm_ros2_control_plugin)"
-      add_gripper="$(arg add_gripper)"/>
-    <!-- Factory gripper. link_eef has to be declared here: upstream puts it in
-         xarm_device_macro.xacro, which we do not include, and lite6.urdf.xacro
-         has its copy commented out. Only the URDF half of the gripper is
-         pulled in; the full uflite_gripper_macro also drags in its own
-         ros2_control system, transmissions and a gazebo grasp-fix plugin, and
-         the finger joint is already declared in our single ros2_control block. -->
-    <xacro:if value="$(arg add_gripper)">
-      <link name="link_eef"/>
-      <joint name="joint_eef" type="fixed">
-        <parent link="link6"/>
-        <child link="link_eef"/>
-        <origin xyz="0 0 0" rpy="0 0 0"/>
-      </joint>
-      <xacro:include filename="$(find xarm_description)/urdf/gripper/uflite_gripper.urdf.xacro"/>
-      <xacro:uflite_gripper_urdf prefix="" attach_to="link_eef"/>
-    </xacro:if>
+      ros2_control_plugin="$(arg arm_ros2_control_plugin)"/>
     <!-- arm base bolted to the top of the mast plate -->
     <joint name="arm_base_joint" type="fixed">
@@ -155,11 +169,4 @@
       <origin xyz="0 0 0.006" rpy="0 0 0"/>
     </joint>
-    <!-- Observation frames for arm avoidance. Massless and geometry-free, so
-         gz lumps them into the parent link and physics is unchanged; they exist
-         only so robot_state_publisher puts them on TF for
-         ammr_wholebody_mpc/arm_detection_points.py. Shared with
-         omni_bot_wholebody.urdf.xacro so both models agree by construction. -->
-    <xacro:include filename="$(find my_omnibot_description)/urdf/arm_detect_points.xacro"/>
-    <xacro:arm_detect_points/>
     <!-- runs a controller_manager inside gz so the 6 arm joints are simulated
          at the physics rate. The base keeps using gz VelocityControl on

Commit message: Auto-update: 2026-09-08 10:48

File: src/my_omnibot_description/urdf/lite6_ros2_control_gz.xacro (robot description, xacro)
@@ -26,9 +26,19 @@
 -->
 <robot xmlns:xacro="http://www.ros.org/wiki/xacro">
+  <!-- All zeros, not the previous tuck.
+       The tuck pose (0, -0.082, 0.089, 0, 1.679, 0) is in self-collision, and
+       not marginally: exact triangle tests put link1 against the gripper shell
+       and against finger2 at 0.000 m, i.e. actually intersecting, with finger1
+       at 1.6 mm. Sampled point clouds had reported 1 to 3 mm there for months
+       because they never landed on the pair of triangles that cross.
+       All zeros clears every non-excluded pair, with link_base to link5 the
+       tightest at 8.79 mm. That is not a lot: joint3 going NEGATIVE from here
+       reaches intersection within 0.05 rad, so any motion starting from this
+       pose needs its direction checked first. -->
   <xacro:property name="tuck_j1" value="0.0"/>
-  <xacro:property name="tuck_j2" value="-0.082"/>
-  <xacro:property name="tuck_j3" value="0.089"/>
+  <xacro:property name="tuck_j2" value="0.0"/>
+  <xacro:property name="tuck_j3" value="0.0"/>
   <xacro:property name="tuck_j4" value="0.0"/>
-  <xacro:property name="tuck_j5" value="1.679"/>
+  <xacro:property name="tuck_j5" value="0.0"/>
   <xacro:property name="tuck_j6" value="0.0"/>
   <xacro:macro name="lite6_ros2_control_gz"

Commit message: Auto-update: 2026-09-08 10:50

File: src/my_omnibot_description/urdf/lite6_ros2_control_gz.xacro (robot description, xacro)
@@ -26,20 +26,16 @@
 -->
 <robot xmlns:xacro="http://www.ros.org/wiki/xacro">
-  <!-- All zeros, not the previous tuck.
-       The tuck pose (0, -0.082, 0.089, 0, 1.679, 0) is in self-collision, and
-       not marginally: exact triangle tests put link1 against the gripper shell
-       and against finger2 at 0.000 m, i.e. actually intersecting, with finger1
-       at 1.6 mm. Sampled point clouds had reported 1 to 3 mm there for months
-       because they never landed on the pair of triangles that cross.
-       All zeros clears every non-excluded pair, with link_base to link5 the
-       tightest at 8.79 mm. That is not a lot: joint3 going NEGATIVE from here
-       reaches intersection within 0.05 rad, so any motion starting from this
-       pose needs its direction checked first. -->
-  <xacro:property name="tuck_j1" value="0.0"/>
-  <xacro:property name="tuck_j2" value="0.0"/>
-  <xacro:property name="tuck_j3" value="0.0"/>
-  <xacro:property name="tuck_j4" value="0.0"/>
-  <xacro:property name="tuck_j5" value="0.0"/>
-  <xacro:property name="tuck_j6" value="0.0"/>
+  <!-- Initial joint angles come from config/arm_initial_pose.yaml, which is
+       the only place they are written. See that file for why they are zeros
+       and for the direction-dependent margin at this pose. -->
+  <xacro:property name="init_pose"
+                  value="${xacro.load_yaml(
+                      '$(find my_omnibot_description)/config/arm_initial_pose.yaml')}"/>
+  <xacro:property name="tuck_j1" value="${init_pose['joint1']}"/>
+  <xacro:property name="tuck_j2" value="${init_pose['joint2']}"/>
+  <xacro:property name="tuck_j3" value="${init_pose['joint3']}"/>
+  <xacro:property name="tuck_j4" value="${init_pose['joint4']}"/>
+  <xacro:property name="tuck_j5" value="${init_pose['joint5']}"/>
+  <xacro:property name="tuck_j6" value="${init_pose['joint6']}"/>
   <xacro:macro name="lite6_ros2_control_gz"
                params="prefix:='' ros2_control_plugin:='gz_ros2_control/GazeboSimSystem'
